Commit message: Update project to match Grad II documentation

File: src/description/urdf/robot.urdf.xacro (robot description, xacro)
@@ -1,8 +1,10 @@
 <?xml version="1.0"?>
-<robot name="sparkx_vehicle" xmlns:xacro="http://www.ros.org/wiki/xacro">
+<robot name="amr_vehicle" xmlns:xacro="http://www.ros.org/wiki/xacro">
   <link name="base_link"/>
   <link name="lidar_link"/>
   <link name="imu_link"/>
   <link name="camera_link"/>
+  <link name="ultrasonic_link"/>
+  <link name="ir_link"/>
   <joint name="base_to_lidar" type="fixed">
     <parent link="base_link"/>
@@ -20,3 +22,13 @@
     <origin xyz="0.25 0.0 0.25" rpy="0 0 0"/>
   </joint>
+  <joint name="base_to_ultrasonic" type="fixed">
+    <parent link="base_link"/>
+    <child link="ultrasonic_link"/>
+    <origin xyz="0.3 0.0 0.05" rpy="0 0 0"/>
+  </joint>
+  <joint name="base_to_ir" type="fixed">
+    <parent link="base_link"/>
+    <child link="ir_link"/>
+    <origin xyz="0.3 0.1 0.05" rpy="0 0 0"/>
+  </joint>
 </robot>

File: src/simulation/urdf/robot.urdf.xacro (robot description, xacro)
@@ -1,120 +1,34 @@
 <?xml version="1.0"?>
-<robot xmlns:xacro="http://www.ros.org/wiki/xacro" name="sparkx_car">
-  <material name="blue"><color rgba="0 0 0.8 1"/></material>
-  <material name="black"><color rgba="0 0 0 1"/></material>
-  <material name="white"><color rgba="1 1 1 1"/></material>
+<robot name="amr_vehicle" xmlns:xacro="http://www.ros.org/wiki/xacro">
   <link name="base_link"/>
-  <joint name="chassis_joint" type="fixed">
-    <parent link="base_link"/>
-    <child link="chassis"/>
-    <origin xyz="0.15 0 0.075" rpy="0 0 0"/>
-  </joint>
-  <link name="chassis">
-    <visual>
-      <origin xyz="0 0 0.025" rpy="0 0 0"/>
-      <geometry><box size="0.3 0.3 0.10"/></geometry>
-      <material name="blue"/>
-    </visual>
-    <collision>
-      <origin xyz="0 0 0.025" rpy="0 0 0"/>
-      <geometry><box size="0.3 0.3 0.10"/></geometry>
-    </collision>
-    <inertial>
-      <origin xyz="0 0 0" rpy="0 0 0"/>
-      <mass value="5.0"/>
-      <inertia ixx="0.05" ixy="0" ixz="0" iyy="0.05" iyz="0" izz="0.08"/>
-    </inertial>
-  </link>
-  <joint name="left_wheel_joint" type="continuous">
-    <parent link="base_link"/>
-    <child link="left_wheel"/>
-    <origin xyz="0 0.175 0.05" rpy="-1.57079632679 0 0"/>
-    <axis xyz="0 0 1"/>
-  </joint>
-  <link name="left_wheel">
-    <visual>
-      <geometry><cylinder radius="0.05" length="0.04"/></geometry>
-      <material name="black"/>
-    </visual>
-    <collision>
-      <geometry><cylinder radius="0.05" length="0.04"/></geometry>
-    </collision>
-    <inertial>
-      <mass value="0.5"/>
-      <inertia ixx="0.001" ixy="0" ixz="0" iyy="0.001" iyz="0" izz="0.001"/>
-    </inertial>
-  </link>
-  <joint name="right_wheel_joint" type="continuous">
-    <parent link="base_link"/>
-    <child link="right_wheel"/>
-    <origin xyz="0 -0.175 0.05" rpy="1.57079632679 0 0"/>
-    <axis xyz="0 0 1"/>
-  </joint>
-  <link name="right_wheel">
-    <visual>
-      <geometry><cylinder radius="0.05" length="0.04"/></geometry>
-      <material name="black"/>
-    </visual>
-    <collision>
-      <geometry><cylinder radius="0.05" length="0.04"/></geometry>
-    </collision>
-    <inertial>
-      <mass value="0.5"/>
-      <inertia ixx="0.001" ixy="0" ixz="0" iyy="0.001" iyz="0" izz="0.001"/>
-    </inertial>
-  </link>
-  <joint name="caster_wheel_joint" type="fixed">
-    <parent link="base_link"/>
-    <child link="caster_wheel"/>
-    <origin xyz="0.25 0 0.025" rpy="0 0 0"/>
-  </joint>
-  <link name="caster_wheel">
-    <visual>
-      <geometry><sphere radius="0.025"/></geometry>
-      <material name="black"/>
-    </visual>
-    <collision>
-      <geometry><sphere radius="0.025"/></geometry>
-    </collision>
-    <inertial>
-      <mass value="0.1"/>
-      <inertia ixx="0.0001" ixy="0" ixz="0" iyy="0.0001" iyz="0" izz="0.0001"/>
-    </inertial>
-  </link>
-  <joint name="lidar_joint" type="fixed">
+  <link name="lidar_link"/>
+  <link name="imu_link"/>
+  <link name="camera_link"/>
+  <link name="ultrasonic_link"/>
+  <link name="ir_link"/>
+  <joint name="base_to_lidar" type="fixed">
     <parent link="base_link"/>
     <child link="lidar_link"/>
-    <origin xyz="0.33 0 0.32" rpy="0 0 0"/>
+    <origin xyz="0.20 0.0 0.20" rpy="0 0 0"/>
   </joint>
-  <link name="lidar_link">
-    <visual>
-      <geometry><cylinder radius="0.05" length="0.04"/></geometry>
-      <material name="black"/>
-    </visual>
-    <collision>
-      <geometry><cylinder radius="0.05" length="0.04"/></geometry>
-    </collision>
-    <inertial>
-      <mass value="0.01"/>
-      <inertia ixx="0.00001" ixy="0" ixz="0" iyy="0.00001" iyz="0" izz="0.00001"/>
-    </inertial>
-  </link>
-  <joint name="imu_joint" type="fixed">
+  <joint name="base_to_imu" type="fixed">
     <parent link="base_link"/>
     <child link="imu_link"/>
-    <origin xyz="0.15 0 0.075" rpy="0 0 0"/>
+    <origin xyz="0.0 0.0 0.10" rpy="0 0 0"/>
   </joint>
-  <link name="imu_link">
-    <visual>
-      <geometry><box size="0.03 0.03 0.02"/></geometry>
-      <material name="white"/>
-    </visual>
-    <collision>
-      <geometry><box size="0.03 0.03 0.02"/></geometry>
-    </collision>
-    <inertial>
-      <mass value="0.02"/>
-      <inertia ixx="0.00001" ixy="0" ixz="0" iyy="0.00001" iyz="0" izz="0.00001"/>
-    </inertial>
-  </link>
+  <joint name="base_to_camera" type="fixed">
+    <parent link="base_link"/>
+    <child link="camera_link"/>
+    <origin xyz="0.25 0.0 0.25" rpy="0 0 0"/>
+  </joint>
+  <joint name="base_to_ultrasonic" type="fixed">
+    <parent link="base_link"/>
+    <child link="ultrasonic_link"/>
+    <origin xyz="0.3 0.0 0.05" rpy="0 0 0"/>
+  </joint>
+  <joint name="base_to_ir" type="fixed">
+    <parent link="base_link"/>
+    <child link="ir_link"/>
+    <origin xyz="0.3 0.1 0.05" rpy="0 0 0"/>
+  </joint>
 </robot>

Commit message: Fix RobotModel missing visual geometries and fix Nav2 out of bounds bug

File: src/description/urdf/robot.urdf.xacro (robot description, xacro)
@@ -1,5 +1,14 @@
 <?xml version="1.0"?>
 <robot name="amr_vehicle" xmlns:xacro="http://www.ros.org/wiki/xacro">
-  <link name="base_link"/>
+  <link name="base_link">
+    <visual>
+      <geometry>
+        <box size="0.3 0.3 0.1"/>
+      </geometry>
+      <material name="blue">
+        <color rgba="0.0 0.0 0.8 1.0"/>
+      </material>
+    </visual>
+  </link>
   <link name="lidar_link"/>
   <link name="imu_link"/>
