Commit message: simulation: complete phase1 task1.2 tf and robot description alignment

File: src/simulation/urdf/robot.urdf.xacro (robot description, xacro)
@@ -1,136 +1,138 @@
 <?xml version="1.0"?>
 <robot xmlns:xacro="http://www.ros.org/wiki/xacro" name="sparkx_car">
-    <material name="blue"><color rgba="0 0 0.8 1"/></material>
-    <material name="black"><color rgba="0 0 0 1"/></material>
-    <material name="white"><color rgba="1 1 1 1"/></material>
-    <link name="base_link"/>
-    <joint name="chassis_joint" type="fixed">
-        <parent link="base_link"/>
-        <child link="chassis"/>
-        <origin xyz="-0.1 0 0"/>
-    </joint>
-    <link name="chassis">
-        <visual>
-            <origin xyz="0.15 0 0.075"/>
-            <geometry><box size="0.3 0.3 0.15"/></geometry>
-            <material name="blue"/>
-        </visual>
-        <collision>
-            <origin xyz="0.15 0 0.075"/>
-            <geometry><box size="0.3 0.3 0.15"/></geometry>
-        </collision>
-        <inertial>
-            <origin xyz="0.15 0 0.075" rpy="0 0 0"/>
-            <mass value="0.5"/>
-            <inertia ixx="0.0046" ixy="0" ixz="0" iyy="0.0046" iyz="0" izz="0.0075"/>
-        </inertial>
-    </link>
-    <joint name="left_wheel_joint" type="continuous">
-        <parent link="base_link"/>
-        <child link="left_wheel"/>
-        <origin xyz="0 0.175 0" rpy="-${pi/2} 0 0"/>
-        <axis xyz="0 0 1"/>
-    </joint>
-    <link name="left_wheel">
-        <visual>
-            <geometry><cylinder radius="0.05" length="0.04"/></geometry>
-            <material name="black"/>
-        </visual>
-        <collision>
-            <geometry><cylinder radius="0.05" length="0.04"/></geometry>
-        </collision>
-        <inertial>
-            <mass value="0.1"/>
-            <inertia ixx="0.00007" ixy="0" ixz="0" iyy="0.00007" iyz="0" izz="0.00012"/>
-        </inertial>
-    </link>
-    <joint name="right_wheel_joint" type="continuous">
-        <parent link="base_link"/>
-        <child link="right_wheel"/>
-        <origin xyz="0 -0.175 0" rpy="${pi/2} 0 0"/>
-        <axis xyz="0 0 1"/>
-    </joint>
-    <link name="right_wheel">
-        <visual>
-            <geometry><cylinder radius="0.05" length="0.04"/></geometry>
-            <material name="black"/>
-        </visual>
-        <collision>
-            <geometry><cylinder radius="0.05" length="0.04"/></geometry>
-        </collision>
-        <inertial>
-            <mass value="0.1"/>
-            <inertia ixx="0.00007" ixy="0" ixz="0" iyy="0.00007" iyz="0" izz="0.00012"/>
-        </inertial>
-    </link>
-    <joint name="caster_wheel_joint" type="fixed">
-        <parent link="chassis"/>
-        <child link="caster_wheel"/>
-        <origin xyz="0.24 0 0"/>
-    </joint>
-    <link name="caster_wheel">
-        <visual>
-            <geometry><sphere radius="0.05"/></geometry>
-            <material name="black"/>
-        </visual>
-        <collision>
-            <geometry><sphere radius="0.05"/></geometry>
-        </collision>
-        <inertial>
-            <mass value="0.1"/>
-            <inertia ixx="0.0001" ixy="0" ixz="0" iyy="0.0001" iyz="0" izz="0.0001"/>
-        </inertial>
-    </link>
-    <joint name="lidar_joint" type="fixed">
-        <parent link="chassis"/>
-        <child link="lidar_link"/>
-        <origin xyz="0.1 0 0.175" rpy="0 0 0"/>
-    </joint>
-    <link name="lidar_link">
-        <visual>
-            <geometry><cylinder radius="0.05" length="0.04"/></geometry>
-            <material name="black"/>
-        </visual>
-        <collision>
-            <geometry><cylinder radius="0.05" length="0.04"/></geometry>
-        </collision>
-        <inertial>
-            <mass value="0.1"/>
-            <inertia ixx="0.0001" ixy="0" ixz="0" iyy="0.0001" iyz="0" izz="0.0001"/>
-        </inertial>
-    </link>
-<gazebo reference="lidar_link">
-  <sensor name="lidar" type="lidar">
-    <always_on>true</always_on>
-    <pose>0 0 0 0 0 0</pose>
-    <visualize>true</visualize>
-    <update_rate>10</update_rate>
-    <topic>scan</topic>
-    <lidar>
-      <scan>
-        <horizontal>
-          <samples>360</samples>
-          <resolution>1</resolution>
-          <min_angle>-3.14159</min_angle>
-          <max_angle>3.14159</max_angle>
-        </horizontal>
-      </scan>
-      <range>
-        <min>0.3</min>
-        <max>12.0</max>
-        <resolution>0.01</resolution>
-      </range>
-    </lidar>
-  </sensor>
-</gazebo>
-    <gazebo>
-        <plugin name="gz::sim::systems::DiffDrive" filename="gz-sim-diff-drive-system">
-            <left_joint>left_wheel_joint</left_joint>
-            <right_joint>right_wheel_joint</right_joint>
-            <wheel_separation>0.35</wheel_separation>
-            <wheel_radius>0.05</wheel_radius>
-            <odom_publish_frequency>30</odom_publish_frequency>
-            <topic>cmd_vel</topic>
-        </plugin>
-    </gazebo>
+  <material name="blue"><color rgba="0 0 0.8 1"/></material>
+  <material name="black"><color rgba="0 0 0 1"/></material>
+  <material name="white"><color rgba="1 1 1 1"/></material>
+  <link name="base_link"/>
+  <joint name="chassis_joint" type="fixed">
+    <parent link="base_link"/>
+    <child link="chassis"/>
+    <origin xyz="-0.1 0 0" rpy="0 0 0"/>
+  </joint>
+  <link name="chassis">
+    <visual>
+      <origin xyz="0.15 0 0.075" rpy="0 0 0"/>
+      <geometry><box size="0.3 0.3 0.15"/></geometry>
+      <material name="blue"/>
+    </visual>
+    <collision>
+      <origin xyz="0.15 0 0.075" rpy="0 0 0"/>
+      <geometry><box size="0.3 0.3 0.15"/></geometry>
+    </collision>
+    <inertial>
+      <origin xyz="0.15 0 0.075" rpy="0 0 0"/>
+      <mass value="0.5"/>
+      <inertia ixx="0.0046" ixy="0" ixz="0" iyy="0.0046" iyz="0" izz="0.0075"/>
+    </inertial>
+  </link>
+  <joint name="left_wheel_joint" type="continuous">
+    <parent link="base_link"/>
+    <child link="left_wheel"/>
+    <origin xyz="0 0.175 0" rpy="-1.57079632679 0 0"/>
+    <axis xyz="0 0 1"/>
+  </joint>
+  <link name="left_wheel">
+    <visual>
+      <geometry><cylinder radius="0.05" length="0.04"/></geometry>
+      <material name="black"/>
+    </visual>
+    <collision>
+      <geometry><cylinder radius="0.05" length="0.04"/></geometry>
+    </collision>
+    <inertial>
+      <mass value="0.1"/>
+      <inertia ixx="0.00007" ixy="0" ixz="0" iyy="0.00007" iyz="0" izz="0.00012"/>
+    </inertial>
+  </link>
+  <joint name="right_wheel_joint" type="continuous">
+    <parent link="base_link"/>
+    <child link="right_wheel"/>
+    <origin xyz="0 -0.175 0" rpy="1.57079632679 0 0"/>
+    <axis xyz="0 0 1"/>
+  </joint>
+  <link name="right_wheel">
+    <visual>
+      <geometry><cylinder radius="0.05" length="0.04"/></geometry>
+      <material name="black"/>
+    </visual>
+    <collision>
+      <geometry><cylinder radius="0.05" length="0.04"/></geometry>
+    </collision>
+    <inertial>
+      <mass value="0.1"/>
+      <inertia ixx="0.00007" ixy="0" ixz="0" iyy="0.00007" iyz="0" izz="0.00012"/>
+    </inertial>
+  </link>
+  <joint name="caster_wheel_joint" type="fixed">
+    <parent link="chassis"/>
+    <child link="caster_wheel"/>
+    <origin xyz="0.24 0 0" rpy="0 0 0"/>
+  </joint>
+  <link name="caster_wheel">
+    <visual>
+      <geometry><sphere radius="0.05"/></geometry>
+      <material name="black"/>
+    </visual>
+    <collision>
+      <geometry><sphere radius="0.05"/></geometry>
+    </collision>
+    <inertial>
+      <mass value="0.1"/>
+      <inertia ixx="0.0001" ixy="0" ixz="0" iyy="0.0001" iyz="0" izz="0.0001"/>
+    </inertial>
+  </link>
+  <joint name="lidar_joint" type="fixed">
+    <parent link="chassis"/>
+    <child link="lidar_link"/>
+    <origin xyz="0.1 0 0.175" rpy="0 0 0"/>
+  </joint>
+  <link name="lidar_link">
+    <visual>
+      <geometry><cylinder radius="0.05" length="0.04"/></geometry>
+      <material name="black"/>
+    </visual>
+    <collision>
+      <geometry><cylinder radius="0.05" length="0.04"/></geometry>
+    </collision>
+    <inertial>
+      <mass value="0.1"/>
+      <inertia ixx="0.0001" ixy="0" ixz="0" iyy="0.0001" iyz="0" izz="0.0001"/>
+    </inertial>
+  </link>
+  <joint name="imu_joint" type="fixed">
+    <parent link="chassis"/>
+    <child link="imu_link"/>
+    <origin xyz="0.0 0.0 0.10" rpy="0 0 0"/>
+  </joint>
+  <link name="imu_link">
+    <visual>
+      <geometry><box size="0.03 0.03 0.02"/></geometry>
+      <material name="white"/>
+    </visual>
+    <collision>
+      <geometry><box size="0.03 0.03 0.02"/></geometry>
+    </collision>
+    <inertial>
+      <mass value="0.02"/>
+      <inertia ixx="0.00001" ixy="0" ixz="0" iyy="0.00001" iyz="0" izz="0.00001"/>
+    </inertial>
+  </link>
+  <joint name="camera_joint" type="fixed">
+    <parent link="chassis"/>
+    <child link="camera_link"/>
+    <origin xyz="0.18 0.0 0.14" rpy="0 0 0"/>
+  </joint>
+  <link name="camera_link">
+    <visual>
+      <geometry><box size="0.04 0.04 0.03"/></geometry>
+      <material name="white"/>
+    </visual>
+    <collision>
+      <geometry><box size="0.04 0.04 0.03"/></geometry>
+    </collision>
+    <inertial>
+      <mass value="0.03"/>
+      <inertia ixx="0.00001" ixy="0" ixz="0" iyy="0.00001" iyz="0" izz="0.00001"/>
+    </inertial>
+  </link>
 </robot>

Commit message: Robot taking targets, moving towards it, gazebo works, rviz2 works, needs to avoid obstacles better

File: src/simulation/urdf/robot.urdf.xacro (robot description, xacro)
@@ -8,20 +8,20 @@
     <parent link="base_link"/>
     <child link="chassis"/>
-    <origin xyz="-0.1 0 0" rpy="0 0 0"/>
+    <origin xyz="0.15 0 0.075" rpy="0 0 0"/>
   </joint>
   <link name="chassis">
     <visual>
-      <origin xyz="0.15 0 0.075" rpy="0 0 0"/>
-      <geometry><box size="0.3 0.3 0.15"/></geometry>
+      <origin xyz="0 0 0.025" rpy="0 0 0"/>
+      <geometry><box size="0.3 0.3 0.10"/></geometry>
       <material name="blue"/>
     </visual>
     <collision>
-      <origin xyz="0.15 0 0.075" rpy="0 0 0"/>
-      <geometry><box size="0.3 0.3 0.15"/></geometry>
+      <origin xyz="0 0 0.025" rpy="0 0 0"/>
+      <geometry><box size="0.3 0.3 0.10"/></geometry>
     </collision>
     <inertial>
-      <origin xyz="0.15 0 0.075" rpy="0 0 0"/>
-      <mass value="0.5"/>
-      <inertia ixx="0.0046" ixy="0" ixz="0" iyy="0.0046" iyz="0" izz="0.0075"/>
+      <origin xyz="0 0 0" rpy="0 0 0"/>
+      <mass value="5.0"/>
+      <inertia ixx="0.05" ixy="0" ixz="0" iyy="0.05" iyz="0" izz="0.08"/>
     </inertial>
   </link>
@@ -29,5 +29,5 @@
     <parent link="base_link"/>
     <child link="left_wheel"/>
-    <origin xyz="0 0.175 0" rpy="-1.57079632679 0 0"/>
+    <origin xyz="0 0.175 0.05" rpy="-1.57079632679 0 0"/>
     <axis xyz="0 0 1"/>
   </joint>
@@ -41,6 +41,6 @@
     </collision>
     <inertial>
-      <mass value="0.1"/>
-      <inertia ixx="0.00007" ixy="0" ixz="0" iyy="0.00007" iyz="0" izz="0.00012"/>
+      <mass value="0.5"/>
+      <inertia ixx="0.001" ixy="0" ixz="0" iyy="0.001" iyz="0" izz="0.001"/>
     </inertial>
   </link>
@@ -48,5 +48,5 @@
     <parent link="base_link"/>
     <child link="right_wheel"/>
-    <origin xyz="0 -0.175 0" rpy="1.57079632679 0 0"/>
+    <origin xyz="0 -0.175 0.05" rpy="1.57079632679 0 0"/>
     <axis xyz="0 0 1"/>
   </joint>
@@ -60,20 +60,20 @@
     </collision>
     <inertial>
-      <mass value="0.1"/>
-      <inertia ixx="0.00007" ixy="0" ixz="0" iyy="0.00007" iyz="0" izz="0.00012"/>
+      <mass value="0.5"/>
+      <inertia ixx="0.001" ixy="0" ixz="0" iyy="0.001" iyz="0" izz="0.001"/>
     </inertial>
   </link>
   <joint name="caster_wheel_joint" type="fixed">
-    <parent link="chassis"/>
+    <parent link="base_link"/>
     <child link="caster_wheel"/>
-    <origin xyz="0.24 0 0" rpy="0 0 0"/>
+    <origin xyz="0.25 0 0.025" rpy="0 0 0"/>
   </joint>
   <link name="caster_wheel">
     <visual>
-      <geometry><sphere radius="0.05"/></geometry>
+      <geometry><sphere radius="0.025"/></geometry>
       <material name="black"/>
     </visual>
     <collision>
-      <geometry><sphere radius="0.05"/></geometry>
+      <geometry><sphere radius="0.025"/></geometry>
     </collision>
     <inertial>
@@ -83,7 +83,7 @@
   </link>
   <joint name="lidar_joint" type="fixed">
-    <parent link="chassis"/>
+    <parent link="base_link"/>
     <child link="lidar_link"/>
-    <origin xyz="0.1 0 0.175" rpy="0 0 0"/>
+    <origin xyz="0.33 0 0.32" rpy="0 0 0"/>
   </joint>
   <link name="lidar_link">
@@ -96,12 +96,12 @@
     </collision>
     <inertial>
-      <mass value="0.1"/>
-      <inertia ixx="0.0001" ixy="0" ixz="0" iyy="0.0001" iyz="0" izz="0.0001"/>
+      <mass value="0.01"/>
+      <inertia ixx="0.00001" ixy="0" ixz="0" iyy="0.00001" iyz="0" izz="0.00001"/>
     </inertial>
   </link>
   <joint name="imu_joint" type="fixed">
-    <parent link="chassis"/>
+    <parent link="base_link"/>
     <child link="imu_link"/>
-    <origin xyz="0.0 0.0 0.10" rpy="0 0 0"/>
+    <origin xyz="0.15 0 0.075" rpy="0 0 0"/>
   </joint>
   <link name="imu_link">
@@ -118,21 +118,3 @@
     </inertial>
   </link>
-  <joint name="camera_joint" type="fixed">
-    <parent link="chassis"/>
-    <child link="camera_link"/>
-    <origin xyz="0.18 0.0 0.14" rpy="0 0 0"/>
-  </joint>
-  <link name="camera_link">
-    <visual>
-      <geometry><box size="0.04 0.04 0.03"/></geometry>
-      <material name="white"/>
-    </visual>
-    <collision>
-      <geometry><box size="0.04 0.04 0.03"/></geometry>
-    </collision>
-    <inertial>
-      <mass value="0.03"/>
-      <inertia ixx="0.00001" ixy="0" ixz="0" iyy="0.00001" iyz="0" izz="0.00001"/>
-    </inertial>
-  </link>
 </robot>

Commit message: Simulation ready v0.1

File: src/simulation/urdf/robot.urdf.xacro (robot description, xacro)
@@ -1,5 +1,10 @@
 <?xml version="1.0"?>
 <robot name="amr_vehicle" xmlns:xacro="http://www.ros.org/wiki/xacro">
+  <!-- Model origin (matches Gazebo model frame, child of odom) -->
   <link name="base_link">
+    <!-- Optional: a small dummy visual so we can see the exact origin in RViz if needed, but usually empty -->
+  </link>
+  <!-- Chassis Visual Link -->
+  <link name="chassis_link">
     <visual>
       <geometry>
@@ -9,35 +14,127 @@
         <color rgba="0.0 0.0 0.8 1.0"/>
       </material>
+      <!-- Visual offset: base_link->chassis_link is 0.15, 0, 0.075. Visual offset in SDF is 0, 0, 0.025 -->
+      <origin xyz="0 0 0.025" rpy="0 0 0"/>
     </visual>
   </link>
-  <link name="lidar_link"/>
-  <link name="imu_link"/>
-  <link name="camera_link"/>
-  <link name="ultrasonic_link"/>
-  <link name="ir_link"/>
+  <joint name="base_to_chassis" type="fixed">
+    <parent link="base_link"/>
+    <child link="chassis_link"/>
+    <origin xyz="0.15 0.0 0.075" rpy="0 0 0"/>
+  </joint>
+  <!-- Wheels -->
+  <link name="left_wheel">
+    <visual>
+      <geometry>
+        <cylinder radius="0.05" length="0.04"/>
+      </geometry>
+      <material name="black">
+        <color rgba="0.1 0.1 0.1 1.0"/>
+      </material>
+    </visual>
+  </link>
+  <joint name="base_to_left_wheel" type="continuous">
+    <parent link="base_link"/>
+    <child link="left_wheel"/>
+    <origin xyz="0 0.175 0.05" rpy="-1.5708 0 0"/>
+    <axis xyz="0 0 1"/>
+  </joint>
+  <link name="right_wheel">
+    <visual>
+      <geometry>
+        <cylinder radius="0.05" length="0.04"/>
+      </geometry>
+      <material name="black">
+        <color rgba="0.1 0.1 0.1 1.0"/>
+      </material>
+    </visual>
+  </link>
+  <joint name="base_to_right_wheel" type="continuous">
+    <parent link="base_link"/>
+    <child link="right_wheel"/>
+    <origin xyz="0 -0.175 0.05" rpy="1.5708 0 0"/>
+    <axis xyz="0 0 1"/>
+  </joint>
+  <link name="caster_wheel">
+    <visual>
+      <geometry>
+        <sphere radius="0.025"/>
+      </geometry>
+      <material name="grey">
+        <color rgba="0.5 0.5 0.5 1.0"/>
+      </material>
+    </visual>
+  </link>
+  <joint name="base_to_caster" type="fixed">
+    <parent link="base_link"/>
+    <child link="caster_wheel"/>
+    <origin xyz="0.25 0.0 0.025" rpy="0 0 0"/>
+  </joint>
+  <!-- Sensors -->
+  <link name="lidar_link">
+    <visual>
+      <geometry>
+        <cylinder radius="0.03" length="0.04"/>
+      </geometry>
+      <material name="red">
+        <color rgba="1.0 0.0 0.0 1.0"/>
+      </material>
+    </visual>
+  </link>
   <joint name="base_to_lidar" type="fixed">
     <parent link="base_link"/>
     <child link="lidar_link"/>
-    <origin xyz="0.20 0.0 0.20" rpy="0 0 0"/>
+    <origin xyz="0.33 0.0 0.32" rpy="0 0 0"/>
   </joint>
+  <link name="camera_link">
+    <visual>
+      <geometry>
+        <box size="0.02 0.05 0.02"/>
+      </geometry>
+      <material name="green">
+        <color rgba="0.0 1.0 0.0 1.0"/>
+      </material>
+    </visual>
+  </link>
+  <joint name="base_to_camera" type="fixed">
+    <parent link="base_link"/>
+    <child link="camera_link"/>
+    <origin xyz="0.40 0.0 0.325" rpy="0 0 0"/>
+  </joint>
+  <link name="ultrasonic_link">
+    <visual>
+      <geometry>
+        <box size="0.02 0.02 0.02"/>
+      </geometry>
+      <material name="yellow">
+        <color rgba="1.0 1.0 0.0 1.0"/>
+      </material>
+    </visual>
+  </link>
+  <joint name="base_to_ultrasonic" type="fixed">
+    <parent link="base_link"/>
+    <child link="ultrasonic_link"/>
+    <origin xyz="0.45 0.0 0.125" rpy="0 0 0"/>
+  </joint>
+  <link name="ir_link">
+    <visual>
+      <geometry>
+        <box size="0.01 0.01 0.01"/>
+      </geometry>
+      <material name="white">
+        <color rgba="1.0 1.0 1.0 1.0"/>
+      </material>
+    </visual>
+  </link>
+  <joint name="base_to_ir" type="fixed">
+    <parent link="base_link"/>
+    <child link="ir_link"/>
+    <origin xyz="0.45 0.1 0.125" rpy="0 0 0"/>
+  </joint>
+  <link name="imu_link"/>
   <joint name="base_to_imu" type="fixed">
     <parent link="base_link"/>
     <child link="imu_link"/>
-    <origin xyz="0.0 0.0 0.10" rpy="0 0 0"/>
-  </joint>
-  <joint name="base_to_camera" type="fixed">
-    <parent link="base_link"/>
-    <child link="camera_link"/>
-    <origin xyz="0.25 0.0 0.25" rpy="0 0 0"/>
-  </joint>
-  <joint name="base_to_ultrasonic" type="fixed">
-    <parent link="base_link"/>
-    <child link="ultrasonic_link"/>
-    <origin xyz="0.3 0.0 0.05" rpy="0 0 0"/>
-  </joint>
-  <joint name="base_to_ir" type="fixed">
-    <parent link="base_link"/>
-    <child link="ir_link"/>
-    <origin xyz="0.3 0.1 0.05" rpy="0 0 0"/>
+    <origin xyz="0.15 0.0 0.075" rpy="0 0 0"/>
   </joint>
 </robot>
